File: PCB/TVP5147M1_decoder/TVP5147M1_decoder.kicad_sch (KiCad schematic)
At the start: 77 parts, among them J1 Conn_02x05_Odd_Even, J2 Conn_02x05_Odd_Even, J3 Conn_02x05_Odd_Even, J4 Conn_02x01, J5 Conn_01x03_Pin, U1 AMS1117-1.8, U2 TVP5147M1IPFP, Y1 14.31818 MHz

Commit message: decoder pcb almost done
Parts:
- removed C28, C29, C31, C32, C33, C34, C35, C36: 0.1uF, Capacitor_SMD:C_1206_3216Metric_Pad1.33x1.80mm_HandSolder, symbol Device:C
- removed CVBS10, CVBS2, CVBS3, CVBS5, CVBS6, CVBS7, CVBS9: Conn_01x02, Connector_PinHeader_2.00mm:PinHeader_1x02_P2.00mm_Vertical, symbol Connector_Generic:Conn_01x02
- removed CVBS8: Conn_Coaxial, Connector_PinHeader_2.00mm:PinHeader_1x02_P2.00mm_Vertical, symbol Connector_Generic:Conn_01x02
- removed J3: Conn_02x05_Odd_Even, Connector_PinHeader_2.54mm:PinHeader_2x05_P2.54mm_Vertical, symbol Connector_Generic:Conn_02x05_Odd_Even
- removed R10, R11, R12, R13, R14, R7, R9: 75Ohm, PCM_Resistor_SMD_AKL:R_0603_1608Metric_Pad1.05x0.95mm_HandSolder, symbol Device:R
- removed R16_BAh1: 10kOhm, PCM_Resistor_SMD_AKL:R_0603_1608Metric_Pad1.05x0.95mm_HandSolder, symbol Device:R
- added D1: LED_3mm, LED_THT:LED_D3.0mm, symbol PCM_SL_Devices:LED_3mm
- added J2, J3: Conn_02x01, Connector_PinHeader_2.54mm:PinHeader_2x01_P2.54mm_Vertical, symbol Connector_Generic:Conn_02x01
- added NT1: NetTie_2, NetTie:NetTie-2_SMD_Pad0.5mm, symbol Device:NetTie_2
- C27, C30: footprint Capacitor_SMD:C_1206_3216Metric_Pad1.33x1.80mm_HandSolder -> Capacitor_SMD:C_0603_1608Metric_Pad1.08x0.95mm_HandSolder
- R6: value 75Ohm -> 5k
- renumbered CVBS4 to CVBS2, J2 to J4, J4 to J5, J5 to J6, R17_B8h1 to RB8
Connections:
- net CVBS_VI_1_B is gone; now on net GND: U2.1 (VI_1_B)
- net CVBS_VI_1_C is gone; now on net GND: U2.2 (VI_1_C)
- net CVBS_VI_2_C is gone; now on net GND: U2.9 (VI_2_C)
- net CVBS_VI_3_A is gone; now on net GND: U2.16 (VI_3_A)
- net CVBS_VI_3_B is gone; now on net GND: U2.17 (VI_3_B)
- net CVBS_VI_3_C is gone; now on net GND: U2.18 (VI_3_C)
- net CVBS_VI_4_A is gone; now on net GND: U2.23 (VI_4_A)
- net +3.3V: now also D1.2
- net CVBS_VI_2_B: now also C30.1
- net GND: now also J1.10 (Pin_10), U2.7 (VI_2_A), U2.81 (EPAD), J2.1 (Pin_1), J2.2 (Pin_2), J3.1 (Pin_1), J3.2 (Pin_2), NT1.2; no longer C37.2, C38.2
- net at R6.1: now also D1.1
- net C0: no longer names the net of U2.70 (C_0/GPIO0)
- net C2: no longer names the net of U2.66 (C_2/GPIO2)
- net C3: no longer names the net of U2.65 (C_3/GPIO3)
- net C4: no longer names the net of U2.64 (C_4/GPIO4)
- net C5: no longer names the net of U2.63 (C_5/GPIO5)
- net C6: no longer names the net of U2.60 (C_6/GPIO6)
- net C7: no longer names the net of U2.59 (C_7/GPIO7)
- net C8: no longer names the net of U2.58 (C_8/GPIO8)
- net C9: no longer names the net of U2.57 (C_9/GPIO9)
- removed net CVBS_VI_2_A: C30.1, U2.7 (VI_2_A)
- new net XGND: C37.2, C38.2, NT1.1
- no-connect marks 8 -> 15
Other:
- moved on the sheet: C30, C37, C38, CVBS2, J4, J5, J6, R15, R8, RB8, Y1

Commit message: added basic hash_drbg
Parts:
- removed C3: 33uF, Capacitor_SMD:C_0603_1608Metric_Pad1.08x0.95mm_HandSolder, symbol Device:C
- removed C8: 10uF, Capacitor_SMD:C_0603_1608Metric_Pad1.08x0.95mm_HandSolder, symbol Device:C
- removed J1: Conn_02x05_Odd_Even, Connector_PinHeader_2.54mm:PinHeader_2x05_P2.54mm_Vertical, symbol Connector_Generic:Conn_02x05_Odd_Even
- added C28, C31, C33: 10uF, Capacitor_SMD:CP_Elec_4x5.7, symbol Device:C_Polarized
- added C29, C35, C39: 22uF, Capacitor_SMD:CP_Elec_5x5.7, symbol Device:C_Polarized
- added C41: 33uF, Capacitor_Tantalum_SMD:CP_EIA-3528-15_AVX-H_Pad1.50x2.35mm_HandSolder, symbol Device:C
- added C45: 10uF, Capacitor_Tantalum_SMD:CP_EIA-3216-18_Kemet-A_Pad1.58x1.35mm_HandSolder, symbol Device:C
- added J7: Conn_02x02_Odd_Even, Connector_PinHeader_2.54mm:PinHeader_2x02_P2.54mm_Vertical, symbol Connector_Generic:Conn_02x02_Odd_Even
- added J9: Conn_02x03_Odd_Even, Connector_PinHeader_2.54mm:PinHeader_2x03_P2.54mm_Vertical, symbol Connector_Generic:Conn_02x03_Odd_Even
- added NT3: NetTie_2, NetTie:NetTie-2_THT_Pad1.0mm, symbol Device:NetTie_2
- added U3: AMS1117-1.8, Package_TO_SOT_SMD:SOT-223-3_TabPin2, symbol Regulator_Linear:AMS1117-1.8
- added U5, U7: AMS1117-3.3, Package_TO_SOT_SMD:SOT-223-3_TabPin2, symbol Regulator_Linear:AMS1117-3.3
- C1, C2, C4: footprint Capacitor_SMD:C_0603_1608Metric_Pad1.08x0.95mm_HandSolder -> Capacitor_Tantalum_SMD:CP_EIA-3528-15_AVX-H_Pad1.50x2.35mm_HandSolder
- C10: footprint Capacitor_THT:CP_Radial_D10.0mm_P5.00mm -> Capacitor_SMD:CP_Elec_5x5.7
- C5: footprint Capacitor_THT:CP_Radial_D8.0mm_P3.50mm -> Capacitor_SMD:CP_Elec_4x5.7
- C6, C7, C9: footprint Capacitor_SMD:C_0603_1608Metric_Pad1.08x0.95mm_HandSolder -> Capacitor_Tantalum_SMD:CP_EIA-3216-18_Kemet-A_Pad1.58x1.35mm_HandSolder
- renumbered NT1 to NT2
Connections:
- net A1.8VDD: now also C45.1
- net AVID: now also J7.4 (Pin_4)
- net DATACLK: now also J7.2 (Pin_2)
- net FSS: now also J7.3 (Pin_3)
- net GLCO/I2CA: now also J7.1 (Pin_1)
- net GND: now also C28.2, C29.2, C31.2, C33.2, C35.2, C39.2, C41.2, C45.2, J9.6 (Pin_6), NT3.2, U3.1 (GND), U5.1 (GND), U7.1 (GND); no longer CVBS1.2 (Ext), CVBS2.2 (Ext), R5.2, R8.2
- net INTREQ: now also J9.4 (Pin_4)
- net PWDN: now also J9.1 (Pin_1)
- net RESETB: now also J9.2 (Pin_2)
- net SCL: now also J9.5 (Pin_5)
- net SDA: now also J9.3 (Pin_3)
- net +1.8V renamed +1.8VPD
- net +1.8VPD: no longer FB3.1
- net +3.3V renamed +5V
- net +5V: now also C28.1, C31.1, C33.1, U3.3 (VI), U5.3 (VI), U7.3 (VI); no longer C1.1, C2.1, FB1.1, FB2.1
- new net +1.8VPA: C29.1, C41.1, FB3.1, U3.2 (VO)
- new net +3.3VPA: C1.1, C35.1, FB1.1, U5.2 (VO)
- new net +3.3VPD: C2.1, C39.1, FB2.1, U7.2 (VO)
- new net CGND: CVBS1.2 (Ext), CVBS2.2 (Ext), NT3.1, R5.2, R8.2
Other:
- moved on the sheet: C10, C11, C12, C13, C14, C15, C16, C17, C18, C19, C20, C21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
